File: BadgersHollowSchematic/BadgersHollowSchematic.sch (KiCad schematic (older format))
At the start: 5 parts

Commit message: Schematic start. mcu and oscillator added
Parts:
- removed C100: 10, Capacitor_THT:CP_Axial_L21.0mm_D8.0mm_P28.00mm_Horizontal, symbol Device:C
- removed R2: 200, Resistor_THT:R_Axial_DIN0204_L3.6mm_D1.6mm_P2.54mm_Vertical, symbol Device:R
- removed R3: 300, Resistor_THT:R_Axial_DIN0207_L6.3mm_D2.5mm_P2.54mm_Vertical, symbol Device:R
- removed R4: 400, Resistor_THT:R_Axial_DIN0204_L3.6mm_D1.6mm_P5.08mm_Vertical, symbol Device:R
- added C1, C2: 22pF, Capacitor_SMD:C_1206_3216Metric_Pad1.42x1.75mm_HandSolder, symbol pspice:C
- added SW1: SW_Push, symbol Switch:SW_Push
- added U1: ATmega32U4-AU, Package_QFP:TQFP-44_10x10mm_P0.8mm, symbol MCU_Microchip_ATmega:ATmega32U4-AU
- added Y1: Crystal, Crystal:Crystal_HC49-U_Vertical, symbol Device:Crystal
- R1: value 100 -> 10K; footprint Capacitor_THT:CP_Axial_L21.0mm_D8.0mm_P28.00mm_Horizontal -> Resistor_SMD:R_1206_3216Metric_Pad1.42x1.75mm_HandSolder
Connections:
- net GND: now also C1.2, C2.2, SW1.1
- net Vcc: now reaches R1.1
- net Reset: now reaches R1.2
- net Reset: now also SW1.2, U1.13 (~RESET)
- new net: U1.14 (VCC), U1.34 (VCC)
- new net: U1.15 (GND), U1.23 (GND), U1.35 (GND), U1.43 (GND)
- new net: C1.1, U1.16 (XTAL2), Y1.2
- new net: C2.1, U1.17 (XTAL1), Y1.1
- new net: U1.24 (AVCC), U1.44 (AVCC)
Changed lines of the file:
@@
 EELAYER 30 0
 EELAYER END
-$Descr A4 11693 8268
+$Descr A1 33110 23386
 encoding utf-8
 Sheet 1 1
@@
 $EndDescr
 $Comp
-L Device:R R2
-U 1 1 5F5AC84A
-P 4500 2950
-F 0 "R2" H 4570 2996 50  0000 L CNN
-F 1 "200" H 4570 2905 50  0000 L CNN
-F 2 "Resistor_THT:R_Axial_DIN0204_L3.6mm_D1.6mm_P2.54mm_Vertical" V 4430 2950 50  0001 C CNN
-F 3 "~" H 4500 2950 50  0001 C CNN
-	1    4500 2950
+L MCU_Microchip_ATmega:ATmega32U4-AU U1
+U 1 1 5F60D4EA
+P 2900 2700
+F 0 "U1" H 2900 811 50  0000 C CNN
+F 1 "ATmega32U4-AU" H 2900 720 50  0000 C CNN
+F 2 "Package_QFP:TQFP-44_10x10mm_P0.8mm" H 2900 2700 50  0001 C CIN
+F 3 "http://ww1.microchip.com/downloads/en/DeviceDoc/Atmel-7766-8-bit-AVR-ATmega16U4-32U4_Datasheet.pdf" H 2900 2700 50  0001 C CNN
+	1    2900 2700
+	1    0    0    -1
+$EndComp
+$Comp
+L Device:Crystal Y1
+U 1 1 5F60FD10
+P 1700 1500
+F 0 "Y1" H 1700 1768 50  0000 C CNN
+F 1 "Crystal" H 1700 1677 50  0000 C CNN
+F 2 "Crystal:Crystal_HC49-U_Vertical" H 1700 1500 50  0001 C CNN
+F 3 "https://www.iqdfrequencyproducts.com/products/pn/LFXTAL027945Bulk.pdf" H 1700 1500 50  0001 C CNN
+	1    1700 1500
+	0    1    1    0
+$EndComp
+Wire Wire Line
+	1800 1400 1800 1350
+Wire Wire Line
+	1800 1350 1700 1350
+Wire Wire Line
+	1800 1600 1800 1650
+Wire Wire Line
+	1800 1650 1700 1650
+Connection ~ 1700 1350
+Wire Wire Line
+	1200 1350 1700 1350
+Wire Wire Line
+	1700 1650 1600 1650
+Connection ~ 1700 1650
+Wire Wire Line
+	1400 2150 1600 2150
+Connection ~ 1400 2150
+Wire Wire Line
+	1200 2150 1400 2150
+$Comp
+L pspice:C C1
+U 1 1 5F693B29
+P 1600 1900
+F 0 "C1" H 1778 1946 39  0000 L CNN
+F 1 "22pF" H 1778 1863 50  0000 L CNN
+F 2 "Capacitor_SMD:C_1206_3216Metric_Pad1.42x1.75mm_HandSolder" H 1600 1900 50  0001 C CNN
+F 3 "https://www.iqdfrequencyproducts.com/products/pn/LFXTAL027945Bulk.pdf" H 1600 1900 50  0001 C CNN
+	1    1600 1900
+	1    0    0    -1
+$EndComp
+$Comp
+L pspice:C C2
+U 1 1 5F67FD87
+P 1200 1900
+F 0 "C2" H 1378 1946 39  0000 L CNN
+F 1 "22pF" H 1378 1863 50  0000 L CNN
+F 2 "Capacitor_SMD:C_1206_3216Metric_Pad1.42x1.75mm_HandSolder" H 1200 1900 50  0001 C CNN
+F 3 "https://www.iqdfrequencyproducts.com/products/pn/LFXTAL027945Bulk.pdf" H 1200 1900 50  0001 C CNN
+	1    1200 1900
+	1    0    0    -1
+$EndComp
+$Comp
+L power:GND #PWR?
+U 1 1 5F67F6EF
+P 1400 2150
+F 0 "#PWR?" H 1400 1900 50  0001 C CNN
+F 1 "GND" H 1405 1977 50  0000 C CNN
+F 2 "" H 1400 2150 50  0001 C CNN
+F 3 "" H 1400 2150 50  0001 C CNN
+	1    1400 2150
+	1    0    0    -1
+$EndComp
+Wire Wire Line
+	1200 1350 1200 1650
+Text GLabel 2300 1200 0    50   Input ~ 0
+Reset
+Wire Wire Line
+	1800 1400 2300 1400
+Wire Wire Line
+	1800 1600 2300 1600
+$Comp
+L Switch:SW_Push SW1
+U 1 1 5F6A57AF
+P 800 3050
+F 0 "SW1" H 800 3335 50  0000 C CNN
+F 1 "SW_Push" H 800 3244 50  0000 C CNN
+F 2 "" H 800 3250 50  0001 C CNN
+F 3 "~" H 800 3250 50  0001 C CNN
+	1    800  3050
 	1    0    0    -1
 $EndComp
 $Comp
 L Device:R R1
-U 1 1 5F5ACEBE
-P 4650 2800
-F 0 "R1" V 4857 2800 50  0000 C CNN
-F 1 "100" V 4766 2800 50  0000 C CNN
-F 2 "Capacitor_THT:CP_Axial_L21.0mm_D8.0mm_P28.00mm_Horizontal" V 4580 2800 50  0001 C CNN
-F 3 "~" H 4650 2800 50  0001 C CNN
-	1    4650 2800
-	0    -1   -1   0
-$EndComp
-$Comp
-L Device:R R3
-U 1 1 5F5ACF00
-P 4800 2950
-F 0 "R3" H 4870 2996 50  0000 L CNN
-F 1 "300" H 4870 2905 50  0000 L CNN
-F 2 "Resistor_THT:R_Axial_DIN0207_L6.3mm_D2.5mm_P2.54mm_Vertical" V 4730 2950 50  0001 C CNN
-F 3 "~" H 4800 2950 50  0001 C CNN
-	1    4800 2950
+U 1 1 5F6A608F
+P 1000 2900
+F 0 "R1" H 1070 2946 50  0000 L CNN
+F 1 "10K" H 1070 2855 50  0000 L CNN
+F 2 "Resistor_SMD:R_1206_3216Metric_Pad1.42x1.75mm_HandSolder" V 930 2900 50  0001 C CNN
+F 3 "https://www.mouser.com/datasheet/2/427/rcse3-1761771.pdf" H 1000 2900 50  0001 C CNN
+	1    1000 2900
 	1    0    0    -1
 $EndComp
+Text GLabel 1000 3050 2    50   Input ~ 0
+Reset
 $Comp
-L Device:C C100
-U 1 1 5F5ADC5F
-P 4950 2800
-F 0 "C100" V 4698 2800 50  0000 C CNN
-F 1 "10" V 4789 2800 50  0000 C CNN
-F 2 "Capacitor_THT:CP_Axial_L21.0mm_D8.0mm_P28.00mm_Horizontal" H 4988 2650 50  0001 C CNN
-F 3 "~" H 4950 2800 50  0001 C CNN
-	1    4950 2800
-	0    1    1    0
-$EndComp
-Connection ~ 4800 2800
-$Comp
-L Device:R R4
-U 1 1 5F5AE074
-P 5100 2950
-F 0 "R4" H 5170 2996 50  0000 L CNN
-F 1 "400" H 5170 2905 50  0000 L CNN
-F 2 "Resistor_THT:R_Axial_DIN0204_L3.6mm_D1.6mm_P5.08mm_Vertical" V 5030 2950 50  0001 C CNN
-F 3 "~" H 5100 2950 50  0001 C CNN
-	1    5100 2950
+L power:GND #PWR?
+U 1 1 5F6A6AAC
+P 600 3050
+F 0 "#PWR?" H 600 2800 50  0001 C CNN
+F 1 "GND" H 605 2877 50  0000 C CNN
+F 2 "" H 600 3050 50  0001 C CNN
+F 3 "" H 600 3050 50  0001 C CNN
+	1    600  3050
 	1    0    0    -1
 $EndComp
-Wire Wire Line
-	5100 3100 4800 3100
-Connection ~ 4800 3100
-Wire Wire Line
-	4800 3100 4500 3100
-$Comp
-L power:GND #PWR0101
-U 1 1 5F5AF0CB
-P 4500 3100
-F 0 "#PWR0101" H 4500 2850 50  0001 C CNN
-F 1 "GND" H 4505 2927 50  0000 C CNN
-F 2 "" H 4500 3100 50  0001 C CNN
-F 3 "" H 4500 3100 50  0001 C CNN
-	1    4500 3100
-	1    0    0    -1
-$EndComp
-Connection ~ 4500 3100
+Text GLabel 1000 2750 1    50   Input ~ 0
+Vcc
 $EndSCHEMATC

Commit message: Schematic down. Need to review, and map columns/rows to correct pins
Parts:
- added C10, C11, C12, C13, C14, C15, C16, C17, C18, C19, C20, C21, C22, C23, C24, C25, C26, C27, C28, C5, C6, C7, C8, C9: 0.1uF, Capacitor_SMD:C_0805_2012Metric_Pad1.15x1.40mm_HandSolder, symbol Device:C
- added C3: 1uF, Resistor_SMD:R_1206_3216Metric_Pad1.42x1.75mm_HandSolder, symbol Device:C
- added C4: 10uF, Capacitor_SMD:C_0603_1608Metric_Pad1.05x0.95mm_HandSolder, symbol Device:C
- added D1, D2: 3.6V, Diode_THT:D_DO-41_SOD81_P3.81mm_Vertical_AnodeUp, symbol Device:D_Zener
- added D10, D11, D12, D13, D14, D15, D16, D17, D18, D19, D20, D21, D22, D23, D24, D25, D26, D27, D28, D4, D5, D6, D7, D8, D9: 1N4148, Diode_SMD:D_SOD-323_HandSoldering, symbol Device:D
- added D29, D30, D31, D32, D33, D34, D35, D36, D37, D38, D39, D40, D41, D42, D43, D44, D45, D46, D47, D48, D49, D50, D51, D52: SK6812, LED_SMD:LED_SK6812_PLCC4_5.0x5.0mm_P3.2mm, symbol LED:SK6812
- added D3: PWR LED, LED_SMD:LED_1206_3216Metric_Pad1.42x1.75mm_HandSolder, symbol Device:LED
- added F1: Polyfuse_Small, Fuse:Fuse_1206_3216Metric, symbol Device:Polyfuse_Small
- added J1: usbc_gct, Connector_USB:USB_C_Receptacle_GCT_USB4085, symbol BadgersHollow:usbc_gct
- added J2: AVR-ISP-6, Connector_PinHeader_2.00mm:PinHeader_2x03_P2.00mm_Vertical, symbol Connector:AVR-ISP-6
- added R2, R3: 5.1K, Resistor_SMD:R_1206_3216Metric_Pad1.42x1.75mm_HandSolder, symbol Device:R
- added R4, R5: 22, Resistor_SMD:R_0805_2012Metric_Pad1.15x1.40mm_HandSolder, symbol Device:R
- added R6, R7: 1.5K, Resistor_SMD:R_0805_2012Metric_Pad1.15x1.40mm_HandSolder, symbol Device:R
- added SW10, SW11, SW12, SW13, SW14, SW15, SW16, SW17, SW18, SW19, SW20, SW21, SW22, SW23, SW24, SW25, SW26, SW27, SW3, SW4, SW5, SW6, SW7, SW8, SW9: SW_SPST, Button_Switch_Keyboard:SW_Cherry_MX_1.00u_PCB, symbol Switch:SW_SPST
- added SW2: SW_Push, Button_Switch_THT:SW_PUSH_6mm, symbol Switch:SW_Push
- added SW29: Rotory Encoder, Rotary_Encoder:RotaryEncoder_Alps_EC11E-Switch_Vertical_H20mm, symbol Device:Rotary_Encoder_Switch
- SW1: footprint (none) -> Button_Switch_THT:SW_PUSH_6mm
Connections:
- net Vcc is gone; now on net +5V: R1.1
- net GND: now also U1.15 (GND), U1.23 (GND), U1.35 (GND), U1.43 (GND), U1.5 (UGND), C10.2, C11.2, C12.2, C13.2, C14.2, C15.2, C16.2, C17.2, C18.2, C19.2, C20.2, C21.2, C22.2, C23.2, C24.2, C25.2, C26.2, C27.2, C28.2, C3.2, C4.2, C5.2, C6.2, C7.2, C8.2, C9.2, D1.2 (A), D2.2 (A), D29.1 (VSS), D30.1 (VSS), D31.1 (VSS), D32.1 (VSS), D33.1 (VSS), D34.1 (VSS), D35.1 (VSS), D36.1 (VSS), D37.1 (VSS), D38.1 (VSS), D39.1 (VSS), D40.1 (VSS), D41.1 (VSS), D42.1 (VSS), D43.1 (VSS), D44.1 (VSS), D45.1 (VSS), D46.1 (VSS), D47.1 (VSS), D48.1 (VSS), D49.1 (VSS), D50.1 (VSS), D51.1 (VSS), D52.1 (VSS), D52.4 (DOUT), J1.A1 (GND), J1.A12 (GND), J1.B1 (GND), J1.S1 (SHIELD), R2.1, R3.1, R7.2, SW2.1
- net Reset: now also J2.5 (~RST)
- net +5V: now reaches U1.14 (VCC), U1.34 (VCC)
- net +5V: now also U1.2 (UVCC), U1.24 (AVCC), U1.44 (AVCC), U1.7 (VBUS), C4.1, D3.2 (A), F1.1, J2.2 (VCC), R6.1
- net boot: now reaches U1.25 (PD4)
- net boot: now also SW2.2
- net d-: now reaches U1.3 (D-)
- net d-: now also R4.1
- net d+: now reaches U1.4 (D+)
- net d+: now also R5.2
- net at U1.6 (UCAP): now also C3.1
- new net: J1.A5 (CC1), R2.2
- new net: J1.B5 (CC2), R3.2
- new net: D1.1 (K), J1.A7 (DN1), J1.B7 (DN2), R4.2, R6.2
- new net: D2.1 (K), J1.A6 (DP1), J1.B6 (DP2), R5.1
- new net: D3.1 (K), R7.1
- new net: D4.2 (A), SW3.1 (A)
- new net: D5.2 (A), SW4.1 (A)
- new net: D6.2 (A), SW5.1 (A)
- new net: D7.2 (A), SW6.1 (A)
- new net: D8.2 (A), SW7.1 (A)
- new net: D9.2 (A), SW8.1 (A)
- new net: D10.2 (A), SW9.1 (A)
- new net: D11.2 (A), SW10.1 (A)
- new net: D12.2 (A), SW11.1 (A)
- new net: D13.2 (A), SW12.1 (A)
- new net: D14.2 (A), SW13.1 (A)
- new net: D15.2 (A), SW14.1 (A)
- new net: D16.2 (A), SW15.1 (A)
- new net: D17.2 (A), SW16.1 (A)
- new net: D18.2 (A), SW17.1 (A)
- new net: D19.2 (A), SW18.1 (A)
- new net: D20.2 (A), SW19.1 (A)
- new net: D21.2 (A), SW20.1 (A)
- new net: D22.2 (A), SW21.1 (A)
- new net: D23.2 (A), SW22.1 (A)
- new net: D24.2 (A), SW23.1 (A)
- new net: D25.2 (A), SW24.1 (A)
- new net: D26.2 (A), SW25.1 (A)
- new net: D27.2 (A), SW26.1 (A)
- new net: D28.2 (A), SW27.1 (A)
- new net: C10.1, C11.1, C12.1, C13.1, C14.1, C15.1, C16.1, C17.1, C18.1, C19.1, C20.1, C21.1, C22.1, C23.1, C24.1, C25.1, C26.1, C27.1, C28.1, C5.1, C6.1, C7.1, C8.1, C9.1, D29.3 (VDD), D30.3 (VDD), D31.3 (VDD), D32.3 (VDD), D33.3 (VDD), D34.3 (VDD), D35.3 (VDD), D36.3 (VDD), D37.3 (VDD), D38.3 (VDD), D39.3 (VDD), D40.3 (VDD), D41.3 (VDD), D42.3 (VDD), D43.3 (VDD), D44.3 (VDD), D45.3 (VDD)
- new net: D29.4 (DOUT), D30.2 (DIN)
- new net: D30.4 (DOUT), D31.2 (DIN)
- new net: D31.4 (DOUT), D32.2 (DIN)
- new net: D33.4 (DOUT), D34.2 (DIN)
- new net: D34.4 (DOUT), D35.2 (DIN)
- new net: D35.4 (DOUT), D36.2 (DIN)
- new net: D36.4 (DOUT), D37.2 (DIN)
- new net: D37.4 (DOUT), D38.2 (DIN)
- new net: D38.4 (DOUT), D39.2 (DIN)
- new net: D39.4 (DOUT), D40.2 (DIN)
- new net: D41.4 (DOUT), D42.2 (DIN)
- new net: D42.4 (DOUT), D43.2 (DIN)
- new net: D43.4 (DOUT), D44.2 (DIN)
- new net: D44.4 (DOUT), D45.2 (DIN)
- new net: D45.4 (DOUT), D46.2 (DIN)
- new net: D46.4 (DOUT), D47.2 (DIN)
- new net: D47.4 (DOUT), D48.2 (DIN)
- new net: D49.4 (DOUT), D50.2 (DIN)
- new net: D50.4 (DOUT), D51.2 (DIN)
- new net: D51.4 (DOUT), D52.2 (DIN)
- new net LEDIN: D29.2 (DIN)
- new net MISO: J2.1 (MISO)
- new net MOSI: J2.4 (MOSI)
- new net SCK: J2.3 (SCK)
- new net VCC: F1.2, J1.A4 (VBUS), J1.A9 (VBUS), J1.B4 (VBUS), J1.B9 (VBUS)
- new net col0: SW13.2 (B), SW18.2 (B), SW23.2 (B), SW3.2 (B), SW8.2 (B)
- new net col1: SW14.2 (B), SW19.2 (B), SW24.2 (B), SW4.2 (B), SW9.2 (B)
- new net col2: SW10.2 (B), SW15.2 (B), SW20.2 (B), SW25.2 (B), SW5.2 (B)
- new net col3: SW11.2 (B), SW16.2 (B), SW21.2 (B), SW26.2 (B), SW6.2 (B)
- new net col4: SW12.2 (B), SW17.2 (B), SW22.2 (B), SW27.2 (B), SW7.2 (B)
- new net row0: D4.1 (K), D5.1 (K), D6.1 (K), D7.1 (K), D8.1 (K)
- new net row1: D10.1 (K), D11.1 (K), D12.1 (K), D13.1 (K), D9.1 (K)
- new net row2: D14.1 (K), D15.1 (K), D16.1 (K), D17.1 (K), D18.1 (K)
- new net row3: D19.1 (K), D20.1 (K), D21.1 (K), D22.1 (K), D23.1 (K)
- new net row4: D24.1 (K), D25.1 (K), D26.1 (K), D27.1 (K), D28.1 (K)
- no-connect marks 0 -> 3
Other:
- moved on the sheet: R1, SW1

Commit message: Finished Schematic, needs to be reviewed then moved to layout
Parts:
- removed SW27: SW_SPST, Button_Switch_Keyboard:SW_Cherry_MX_1.00u_PCB, symbol Switch:SW_SPST
- SW27: renamed from SW29; footprint Rotary_Encoder:RotaryEncoder_Alps_EC11E-Switch_Vertical_H20mm -> Rotary_Encoder:RotaryEncoder_Alps_EC11E-Switch_Vertical_H20mm_CircularMountingHoles
Connections:
- net row4 is gone; now on net rer: D24.1 (K), D25.1 (K), D26.1 (K), D27.1 (K), D28.1 (K)
- net GND: now also SW27.C
- net LEDIN: now also U1.28 (PB4)
- net MISO: now also U1.11 (PB3)
- net MOSI: now also U1.10 (PB2)
- net SCK: now also U1.9 (PB1)
- net col0: now also U1.21 (PD3)
- net col1: now also U1.22 (PD5)
- net col2: now also U1.18 (PD0)
- net col3: now also U1.19 (PD1)
- net col4: now also SW27.S1, U1.20 (PD2)
- net row0: now also U1.37 (PF6)
- net row1: now also U1.38 (PF5)
- net row2: now also U1.39 (PF4)
- net row3: now also U1.40 (PF1)
- net rencb: now reaches U1.29 (PB5)
- net rencb: now also SW27.B
- net renca: now reaches U1.30 (PB6)
- net renca: now also SW27.A
- net rer: now reaches U1.41 (PF0)
- net at SW27.S2: now also D28.2 (A)
- no-connect marks 3 -> 12
Other:
- note added: "ATmega32U4-Au\nMCU\n"
- note added: "AVR ISP Connector\n"
- note added: "Boot Switch\n"
- note added: "Power Indicator\n"
- note added: "Reset\n"
- note added: "Rotary Encoder\n"
- note added: "Switch Matrix\n"
- note added: "USB C Connector\n"
- note added: "USB Power Smoothing Cap\n"
- note added: "Underglow RGB LED Chain\n"
- moved on the sheet: C1, C2, C3, C4, D1, D2, D3, F1, J1, J2, R1, R2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

Commit message: Working on layout
Parts:
- removed D17: 1N4148, Diode_SMD:D_SOD-323_HandSoldering, symbol Device:D
- removed SW16: SW_SPST, Button_Switch_Keyboard:SW_Cherry_MX_1.00u_PCB, symbol Switch:SW_SPST
- SW11, SW21: footprint Button_Switch_Keyboard:SW_Cherry_MX_1.00u_PCB -> Button_Switch_Keyboard:SW_Cherry_MX_2.00u_Vertical_PCB
Connections:
- net boot: now also U1.33 (~HWB~/PE2); no longer U1.25 (PD4)
- net col0: now also U1.18 (PD0); no longer U1.21 (PD3)
- net col1: now also U1.19 (PD1); no longer U1.22 (PD5)
- net col2: now also U1.20 (PD2); no longer U1.18 (PD0)
- net col3: now also SW27.S1, U1.21 (PD3); no longer SW26.2 (B), U1.19 (PD1)
- net col4: now also SW26.2 (B), U1.25 (PD4); no longer SW27.S1, U1.20 (PD2)
- no-connect marks 12 -> 14
Other:
- moved on the sheet: D27, SW26
Changed lines of the file:
@@
 	1    0    0    -1
 $EndComp
-Text GLabel 3500 3100 2    50   Input ~ 0
+Text GLabel 3500 3600 2    50   Input ~ 0
 boot
 Text GLabel 1600 6600 2    50   Input ~ 0
@@
 F 0 "SW11" H 14300 2735 50  0000 C CNN
 F 1 "SW_SPST" H 14300 2644 50  0000 C CNN
-F 2 "Button_Switch_Keyboard:SW_Cherry_MX_1.00u_PCB" H 14300 2500 50  0001 C CNN
+F 2 "Button_Switch_Keyboard:SW_Cherry_MX_2.00u_Vertical_PCB" H 14300 2500 50  0001 C CNN
 F 3 "~" H 14300 2500 50  0001 C CNN
 	1    14300 2500
@@
 $EndComp
 $Comp
-L Switch:SW_SPST SW16
-U 1 1 5FA0F031
-P 14300 3100
-F 0 "SW16" H 14300 3335 50  0000 C CNN
-F 1 "SW_SPST" H 14300 3244 50  0000 C CNN
-F 2 "Button_Switch_Keyboard:SW_Cherry_MX_1.00u_PCB" H 14300 3100 50  0001 C CNN
-F 3 "~" H 14300 3100 50  0001 C CNN
-	1    14300 3100
-	1    0    0    -1
-$EndComp
-$Comp
-L Device:D D17
-U 1 1 5FA0F037
-P 14100 3250
-F 0 "D17" V 14146 3170 50  0000 R CNN
-F 1 "1N4148" V 14055 3170 50  0000 R CNN
-F 2 "Diode_SMD:D_SOD-323_HandSoldering" H 14100 3250 50  0001 C CNN
-F 3 "https://www.mouser.com/datasheet/2/115/ds30097-88009.pdf" H 14100 3250 50  0001 C CNN
-	1    14100 3250
-	0    -1   -1   0
-$EndComp
-$Comp
 L Switch:SW_SPST SW17
 U 1 1 5FA0F03D
@@
 F 0 "SW21" H 14300 3935 50  0000 C CNN
 F 1 "SW_SPST" H 14300 3844 50  0000 C CNN
-F 2 "Button_Switch_Keyboard:SW_Cherry_MX_1.00u_PCB" H 14300 3700 50  0001 C CNN
+F 2 "Button_Switch_Keyboard:SW_Cherry_MX_2.00u_Vertical_PCB" H 14300 3700 50  0001 C CNN
 F 3 "~" H 14300 3700 50  0001 C CNN
 	1    14300 3700
@@
 	0    -1   -1   0
 $EndComp
-$Comp
-L Switch:SW_SPST SW26
-U 1 1 5FA474CA
-P 14300 4300
-F 0 "SW26" H 14300 4535 50  0000 C CNN
-F 1 "SW_SPST" H 14300 4444 50  0000 C CNN
-F 2 "Button_Switch_Keyboard:SW_Cherry_MX_1.00u_PCB" H 14300 4300 50  0001 C CNN
-F 3 "~" H 14300 4300 50  0001 C CNN
-	1    14300 4300
-	1    0    0    -1
-$EndComp
-$Comp
-L Device:D D27
-U 1 1 5FA474D0
-P 14100 4450
-F 0 "D27" V 14146 4370 50  0000 R CNN
-F 1 "1N4148" V 14055 4370 50  0000 R CNN
-F 2 "Diode_SMD:D_SOD-323_HandSoldering" H 14100 4450 50  0001 C CNN
-F 3 "https://www.mouser.com/datasheet/2/115/ds30097-88009.pdf" H 14100 4450 50  0001 C CNN
-	1    14100 4450
-	0    -1   -1   0
-$EndComp
 Wire Wire Line
 	12850 1900 12850 2500
@@
 Connection ~ 14500 2500
 Wire Wire Line
-	14500 2500 14500 3100
-Connection ~ 14500 3100
-Wire Wire Line
-	14500 3100 14500 3700
-Connection ~ 14500 3700
-Wire Wire Line
-	14500 3700 14500 4300
-Wire Wire Line
 	15050 1900 15050 2500
 Connection ~ 15050 2500
@@
 Connection ~ 15050 3700
 Wire Wire Line
-	15050 3700 15050 4300
-Wire Wire Line
 	12450 2200 13000 2200
 Connection ~ 13000 2200
@@
 Connection ~ 13550 3400
 Wire Wire Line
-	13550 3400 14100 3400
-Connection ~ 14100 3400
-Wire Wire Line
-	14100 3400 14650 3400
-Wire Wire Line
 	12450 4000 13000 4000
 Connection ~ 13000 4000
@@
 	13000 4600 13550 4600
 Connection ~ 13550 4600
-Wire Wire Line
-	13550 4600 14100 4600
-Connection ~ 14100 4600
-Wire Wire Line
-	14100 4600 14650 4600
 Text GLabel 12850 1500 1    50   Input ~ 0
 col0
@@
 Text Notes 13700 950  0    50   ~ 0
 Switch Matrix\n
-Text GLabel 15050 4300 3    50   Input ~ 0
+Text GLabel 14500 4300 3    50   Input ~ 0
 rec
-Text GLabel 14650 4600 2    50   Input ~ 0
+Text GLabel 14100 4600 1    50   Input ~ 0
 rer
 $Comp
@@
 Text GLabel 3500 3900 2    50   Input ~ 0
 row4
+Text GLabel 3500 2700 2    50   Input ~ 0
+col0
+Text GLabel 3500 2800 2    50   Input ~ 0
+col1
+Text GLabel 3500 2900 2    50   Input ~ 0
+col2
 Text GLabel 3500 3000 2    50   Input ~ 0
-col0
-Text GLabel 3500 3200 2    50   Input ~ 0
-col1
-Text GLabel 3500 2700 2    50   Input ~ 0
-col2
-Text GLabel 3500 2800 2    50   Input ~ 0
 col3
-Text GLabel 3500 2900 2    50   Input ~ 0
+Text GLabel 3500 3100 2    50   Input ~ 0
 col4
 NoConn ~ 3500 3700
-NoConn ~ 3500 3600
 NoConn ~ 3500 4400
 NoConn ~ 3500 3400
@@
 NoConn ~ 3500 2200
 NoConn ~ 3500 1500
+NoConn ~ 9350 2050
+NoConn ~ 3500 3200
+NoConn ~ 12150 3250
+Connection ~ 14500 3700
+Wire Wire Line
+	14500 3700 14500 4300
+$Comp
+L Switch:SW_SPST SW26
+U 1 1 5FA474CA
+P 14850 4300
+F 0 "SW26" H 14850 4535 50  0000 C CNN
+F 1 "SW_SPST" H 14850 4444 50  0000 C CNN
+F 2 "Button_Switch_Keyboard:SW_Cherry_MX_1.00u_PCB" H 14850 4300 50  0001 C CNN
+F 3 "~" H 14850 4300 50  0001 C CNN
+	1    14850 4300
+	1    0    0    -1
+$EndComp
+$Comp
+L Device:D D27
+U 1 1 5FA474D0
+P 14650 4450
+F 0 "D27" V 14696 4370 50  0000 R CNN
+F 1 "1N4148" V 14605 4370 50  0000 R CNN
+F 2 "Diode_SMD:D_SOD-323_HandSoldering" H 14650 4450 50  0001 C CNN
+F 3 "https://www.mouser.com/datasheet/2/115/ds30097-88009.pdf" H 14650 4450 50  0001 C CNN
+	1    14650 4450
+	0    -1   -1   0
+$EndComp
+Wire Wire Line
+	13550 4600 14650 4600
+Wire Wire Line
+	15050 3700 15050 4300
+Wire Wire Line
+	14500 2500 14500 3700
+Wire Wire Line
+	13550 3400 14650 3400
 $EndSCHEMATC

Commit message: Layout done. Now working on routing
Parts:
- removed C10, C13, C16, C19, C22, C25, C28: 0.1uF, Capacitor_SMD:C_0805_2012Metric_Pad1.15x1.40mm_HandSolder, symbol Device:C
- removed D46, D47, D48, D49, D50, D51, D52: SK6812, LED_SMD:LED_SK6812_PLCC4_5.0x5.0mm_P3.2mm, symbol LED:SK6812
Connections:
- net GND: now also D45.4 (DOUT)
