File: BadgersHollowSchematic/BadgersHollowSchematic.sch (KiCad schematic (older format))
At the start: 103 parts, among them J1 usbc_gct, J2 AVR-ISP-6, SW1 SW_Push, SW10 SW_SPST, SW11 SW_SPST, SW12 SW_SPST, SW13 SW_SPST, SW14 SW_SPST, SW15 SW_SPST, SW17 SW_SPST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

Commit message: Final V1 before first test run order
Connections:
- no-connect marks 14 -> 13
Changed lines of the file:
@@
 NoConn ~ 3500 2200
 NoConn ~ 3500 1500
-NoConn ~ 9400 1950
 NoConn ~ 3500 3100
 NoConn ~ 10950 3300
